File: qsd67lc.sch (EAGLE design)
At the start: 0 parts

Commit message: added mountholes added atmega8 (incl. leds, switches)
Parts:
- added C1, C3, C4: (no value), rcl:C-EUC0805
- added H1, H2, H3, H4: MOUNT-HOLE3.0, holes:MOUNT-HOLE3.0
- added IC1: MEGA8-P, atmel:MEGA8-P
- added LED1, LED2, LED3: (no value), led:LEDCHIP-LED0805
- added Q1: (no value), crystal:CRYSTALHC18U-V
- added R1, R2, R3, R4, R5, R6: (no value), rcl:R-EU_R0805
- added S1, S2: (no value), switch-omron:10-XX
- added SV1: (no value), con-harting-ml:ML6
Connections:
- new net +5V: IC1.AREF, IC1.AVCC, IC1.VCC@1, R1.2, SV1.5
- new net DLE: R2.2, R3.2, R4.2, R5.2, R6.2
- new net GND: C1.2, C3.1, C4.1, IC1.GND, IC1.GND@1, SV1.1
- new net MISO: IC1.PB4(MISO), SV1.6
- new net MOSI: IC1.PB3(MOSI/OC2), SV1.3
- new net N$1: IC1.PC1(ADC1), LED2.C
- new net N$10: IC1.PC4(ADC4/SDA), S1.P, S1.P1
- new net N$11: R6.1, S2.S, S2.S1
- new net N$12: IC1.PC5(ADC5/SCL), S2.P, S2.P1
- new net N$2: C3.2, IC1.PB6(XTAL1/TOSC1), Q1.1
- new net N$3: C4.2, IC1.PB7(XTAL2/TOSC2), Q1.2
- new net N$4: LED2.A, R3.1
- new net N$5: LED1.A, R2.1
- new net N$6: LED3.A, R4.1
- new net N$7: IC1.PC0(ADC0), LED1.C
- new net N$8: R5.1, S1.S, S1.S1
- new net N$9: IC1.PC2(ADC2), LED3.C
- new net RESET: C1.1, IC1.PC6(/RESET), R1.1, SV1.2
- new net RXD_5V: IC1.PD0(RXD)
- new net SCK: IC1.PB5(SCK), SV1.4
- new net TXD_5V: IC1.PD1(TXD)
