File: k-line-adapter.brd (EAGLE design)
At the start: 76.2 x 41.6 mm, 22 parts, among them IC3 MAX3232CPE, IC5 LM2576S-5.0, T1 BC847C, X2 RS232

Commit message: working on kline adapter ...
Parts:
- IC3: value MAX3232CPE -> MAX232
Changed lines of the file:
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@@
 <drawing>
 <settings>
-<setting alwaysvectorfont="no"/>
+<setting alwaysvectorfont="yes"/>
 <setting verticaltext="up"/>
 </settings>
@@
 <attribute name="VALUE" x="36.83" y="11.811" size="1.27" layer="27" ratio="10"/>
 </element>
-<element name="IC3" library="maxim" library_urn="urn:adsk.eagle:library:269" package="DIL16" package3d_urn="urn:adsk.eagle:package:922/2" value="MAX3232CPE" x="55.88" y="20.32" smashed="yes" rot="R90">
+<element name="IC3" library="maxim" library_urn="urn:adsk.eagle:library:269" package="DIL16" package3d_urn="urn:adsk.eagle:package:922/2" value="MAX232" x="55.88" y="20.32" smashed="yes" rot="R90">
 <attribute name="MF" value="MAXIM" x="113.03" y="63.5" size="1.778" layer="27" rot="R90" display="off"/>
-<attribute name="MPN" value="MAX3232CPE+" x="113.03" y="63.5" size="1.778" layer="27" rot="R90" display="off"/>
+<attribute name="MPN" value="MAX232ACPE+" x="113.03" y="63.5" size="1.778" layer="27" rot="R90" display="off"/>
 <attribute name="NAME" x="58.801" y="9.779" size="1.27" layer="25" ratio="10" rot="R180"/>
-<attribute name="OC_FARNELL" value="9724494" x="113.03" y="63.5" size="1.778" layer="27" rot="R90" display="off"/>
-<attribute name="OC_NEWARK" value="68K4626" x="113.03" y="63.5" size="1.778" layer="27" rot="R90" display="off"/>
+<attribute name="OC_FARNELL" value="9723773" x="113.03" y="63.5" size="1.778" layer="27" rot="R90" display="off"/>
+<attribute name="OC_NEWARK" value="68K4544" x="113.03" y="63.5" size="1.778" layer="27" rot="R90" display="off"/>
 <attribute name="VALUE" x="56.515" y="12.827" size="1.27" layer="27" ratio="10" rot="R90"/>
 </element>
@@
 </signals>
 <mfgpreviewcolors>
-<mfgpreviewcolor name="soldermaskcolor" color="0xC8008000"/>
+<mfgpreviewcolor name="soldermaskcolor" color="0xC8FF0000"/>
 <mfgpreviewcolor name="silkscreencolor" color="0xFFFEFEFE"/>
-<mfgpreviewcolor name="backgroundcolor" color="0xFF282828"/>
+<mfgpreviewcolor name="backgroundcolor" color="0xFF000000"/>
 <mfgpreviewcolor name="coppercolor" color="0xFFFFBF00"/>
-<mfgpreviewcolor name="substratecolor" color="0xFF786E46"/>
+<mfgpreviewcolor name="substratecolor" color="0xFFAA0000"/>
 </mfgpreviewcolors>
 </board>
