File: k-line-adapter.sch (EAGLE design)
At the start: 22 parts, among them IC3 MAX3232CPE, IC5 LM2576S-5.0, T1 BC847C, X2 RS232

Commit message: working on kline adapter ...
Parts:
- IC3: value MAX3232CPE -> MAX232; device maxim:MAX3232CPE -> maxim:MAX232
Changed lines of the file:
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@@
 </classes>
 <parts>
-<part name="IC3" library="maxim" library_urn="urn:adsk.eagle:library:269" deviceset="MAX3232*" device="PE" package3d_urn="urn:adsk.eagle:package:922/2" technology="C"/>
+<part name="IC3" library="maxim" library_urn="urn:adsk.eagle:library:269" deviceset="MAX232" device="" package3d_urn="urn:adsk.eagle:package:922/2"/>
 <part name="GND7" library="supply1" library_urn="urn:adsk.eagle:library:371" deviceset="GND" device=""/>
 <part name="GND8" library="supply1" library_urn="urn:adsk.eagle:library:371" deviceset="GND" device=""/>
