File: qsd67lc_v2.sch (EAGLE design)
At the start: 67 parts, among them CON1 RIA-AKL-230-04, CON2 RIA-AKL-230-04, CON3 RIA-AKL-230-03, IC1 MEGA8-P, IC2 BTS555E3146, IC3 MAX3232CPE, IC4 LM2576S, IC5 FT232RL, IC6 ISO7221A, Q1 16MHz, T1 BCR141, U1 HC_05, X2 RS232

Commit message: started development of v2 prototype containing OBDII diagnostics capabilities.
Parts:
- removed IC6: ISO7221A, texas:ISO7221A
- removed U2: (no value), MicroUSB:USB""
- removed X2: RS232, con-subd:F09HP
- added D3: PESD1CAN, diode:PESD1CAN
- added D4, D5: BAS40-06, diode:BAS40-06
- added D6: 1N5822, diode:SCHOTTKY-DIODEDO201T15
- added D7: (no value), diode:DIODE-SOD123
- added D8, D9: (no value), diode:ZENER-DIODESMB
- added JP5: (no value), pinhead:PINHD-1X1
- added L2: 100uH, rcl:L-EU2200-15.24
- added LED10, LED12: orange, led:LEDCHIP-LED0805
- added LED11, LED9: yellow, led:LEDCHIP-LED0805
- added LED13, LED8: green, led:LEDCHIP-LED0805
- added Q2: IRLZ44Z, transistor-power:IRLZ44Z
- added Q3: 16MHz, crystal:CRYSTALHC49U70
- added Q4: IRLML5203, transistor-power:IRLML5203
- added R15: 220R, rcl:R-EU_M0805
- added R16, R21, R22, R23, R24, R25: 220R, rcl:R-EU_R0805
- added R17: 10k, rcl:R-EU_R0805
- added R20: 100k, rcl:R-EU_R0805
- added R26, R27, R28: (no value), rcl:R-EU_R0805
- added R5: 1k, rcl:R-EU_R0805
- added S2: RST_NVM, switch-omron:10-XX
- added T2: (no value), transistor:MMBT3906LT1-PNP-SOT23-BEC
- added T3: BCR141S, digital-transistors-2:BCR141S
- added U$1: STN1110-SOIC28, 1zac:STN1110-SOIC28
- added X1: (no value), con-subd:M09HP
- C11, C5, C8: value 100nF -> 1uF
- C13: value 100nF -> 10uF; device rcl:C-EUC0805 -> rcl:CPOL-EUE5-10.5
- C14: value 100nF -> 100uF; device rcl:C-EUC0805 -> rcl:CPOL-EUE5-13
- C15: value 4,7µF -> 1000uF; device rcl:CPOL-EUE2.5-5 -> rcl:CPOL-EUE5-10.5
- C6, C7: value 100nF -> 30pF
- IC3: value MAX3232CPE -> 74AC08D; device maxim:MAX3232CPE -> 74xx-eu:74AC08D
- IC4: value LM2576S -> LM2576S-3.3
- IC5: value FT232RL -> LM2576S-5.0; device ftdichip:FT232RL -> v-reg-3:LM2576S
- JP1: value UART_SELECTOR -> (none); device pinhead:PINHD-2X3 -> pinhead:PINHD-1X3
- LED4: value green -> blue; device led:LEDSML0805 -> led:LEDCHIP-LED0805
- LED5: value orange -> blue; device led:LEDSML0805 -> led:LEDCHIP-LED0805
- R10: value 10k -> 220R; device rcl:R-EU_R0805 -> rcl:R-EU_M0805
- R18: value 270R -> 10R
- R19: value 270R -> 100k
Connections:
- removed net CS: IC1.PB2(SS/OC1B)
- removed net GND_USB: C13.2, C14.2, C15.-, C16.2, C18.1, IC5.GND, IC5.GND@1, IC5.GND@2, IC5.GND@A, IC5.TEST, IC6.GND2, U2.GND
- removed net N$20 (its old number): C7.1, IC3G$1.C1-
- removed net RS232_RX: IC3G$1.T1OUT, X2.3
- removed net RS232_RX_D: IC5.TXD, IC6.INA
- removed net RS232_TX: IC3G$1.R1IN, X2.2
- removed net RS232_TX_D: IC5.RXD, IC6.OUTB
- removed net RXD_RS232: IC3G$1.R1OUT, IC6.OUTA, JP1.5
- removed net TXD_RS232: IC3G$1.T1IN, IC6.INB, JP1.6
- removed net USB_D+: IC5.USBDP, U2.D+
- removed net USB_D-: IC5.USBDM, U2.D-
- removed net USB_RX_LED: IC5.CBUS0, R18.1
- removed net USB_TX_LED: IC5.CBUS1, R19.1
- removed net VCCIO_USB: C14.1, C18.2, IC5.!RESET, IC5.3V3OUT, IC5.VCCIO, IC6.VCC2, LED4.A, LED5.A
- removed net VCC_USB: C13.1, C15.+, C16.1, IC5.VCC, U2.VBUS
- new net !ISO_K_TX: U$1.!ISO_K_TX
- new net !ISO_L_TX: U$1.!ISO_L_TX
- new net !ISO_RX: U$1.!ISO_RX
- new net !J1850_BUS-_TX: U$1.!J1850_BUS-_TX
- new net !OBD_RX_LED: U$1.!OBD_RX_LED/!INT
- new net !OBD_TX_LED: R19.2, S2.S, U$1.!OBD_TX_LED/!RST_NVM
- new net !UART_RX_LED: U$1.!UART_RX_LED
- new net !UART_TX_LED: U$1.!UART_TX_LED
- new net !VPW_RX: U$1.!VPW_RX
- new net +12V_RAW: C17.1, D7.A, JP1.2
- new net +5V: C15.+, IC5.FB, JP5.1, L2.2, LED13.A
- new net ANALOG_IN: U$1.ANALOG_IN
- new net CAN_RX: U$1.CAN_RX
- new net CAN_TX: U$1.CAN_TX
- new net HS_CAN_HI: X1.3
- new net HS_CAN_LO: D3.2, X1.5
- new net J1850_BUS+: D5.K2, X1.7
- new net J1850_BUS+_TX: U$1.J1850_BUS+TX
- new net J1850_BUS-: D5.K1, X1.6
- new net KL15: CON1.P$4, JP1.1
- new net KL30: JP1.3, X1.9
- new net K_LINE: D4.K2, X1.4
- new net L_LINE: D4.K1, X1.8
- new net N$1: C8.1, R17.1, U$1.!RESET
- new net N$10: LED5.C, R15.2
- new net N$21: C11.1, R18.2, U$1.AVDD
- new net N$24: C13.+, U$1.VCAP
- new net N$25: R20.2, U$1.PWR_CTRL
- new net N$27: LED11.A, R22.2
- new net N$28: LED10.A, R23.2
- new net N$29: LED9.A, R24.2
- new net N$30: D6.C, IC5.OUT, L2.1
- new net N$31: LED13.C, R25.2
- new net N$32: D8.C, R26.1, R27.2
- new net N$33: R27.1, T2.B
- new net N$34: C18.1, D9.A, Q4.G, R28.2, T2.C
- new net N$8: LED4.C, R10.2
- new net OBD_RX_LED: LED11.C
- new net OBD_TX_LED: LED12.C
- new net PWM/!VPW: U$1.PWM/!VPW
- new net PWM_RX: U$1.PWM_RX
- new net RXD_OBD: IC3D.O, U$1.UART_RX
- new net TXD_OBD: IC3C.I0, R5.1, U$1.UART_TX
- new net UART_EN_BT: IC1.PD5(T1), IC3A.I1, IC3B.I1, T3A.B
- new net UART_EN_OBD: IC1.PD6(AIN0), IC3C.I1, IC3D.I1, T3B.B
- new net UART_RX_LED: LED9.C
- new net UART_TX_LED: LED10.C
- net +12V: now also C14.+, C16.1, IC5.VIN, Q2.D, Q4.D; no longer CON1.P$4
- net +3V3: now also C5.2, LED8.A, R17.2, R18.1, R19.1, R21.1, R22.1, R23.1, R24.1, R5.2, T3A.C, T3B.C, U$1.VDD; no longer C11.1, C17.2, IC3P.VCC, IC6.VCC1, R10.2
- net 12V_OUT: now also Q2.S
- net GND: now also C13.-, C14.-, C15.-, C16.2, C17.2, C18.2, C5.1, C7.2, C8.2, D3.1, D3.3, D4.AA, D5.AA, D6.A, D8.A, IC5.GND, IC5.OFF, R10.1, R15.1, R16.1, R20.1, R25.1, R28.1, S2.P, SV1.6, U$1.AVSS, U$1.VSS@1, U$1.VSS@2, X1.1, X1.2; no longer C17.1, C5.2, IC3P.GND, IC6.GND1, SV1.1, X2.1, X2.5
- net MISO: now also SV1.1; no longer SV1.6
- net MOSI: now also SV1.4; no longer SV1.3
- net N$11: now also LED8.C, R16.2; no longer C5.1, IC3G$1.V+
- net N$15: now also LED4.A, T3A.E; no longer C6.1, IC3G$1.V-
- net N$16: now also Q2.G
- net N$17: now also LED5.A, T3B.E; no longer C7.2, IC3G$1.C1+
- net N$18: now also C7.1, Q3.2, U$1.OSC1; no longer C8.2, IC3G$1.C2+
- net N$19: now also D7.C, D9.C, Q4.S, R26.2, T2.E; no longer C8.1, IC3G$1.C2-
- net N$23: now also C6.1, Q3.1, U$1.OSC2; no longer LED4.C, R18.2
- net N$26: now also LED12.A, R21.2; no longer LED5.C, R19.2
- net PAIRED_STATE: now also IC1.PD4(XCK/T0)
- net QS+: no longer R10.1
- net RESET: now also SV1.5; no longer SV1.2
- net RXD: now also IC3A.O, IC3C.O; no longer JP1.3
- net RXD_BT: now also IC3B.O; no longer JP1.1
- net SCK: now also SV1.3; no longer SV1.4
- net TXD: now also IC3B.I0, IC3D.I0; no longer JP1.4
- net TXD_BT: now also IC3A.I0; no longer JP1.2
Other:
- note added: "OBD II"
- note added: "alternative mounting"
- note added: "bluetooth"
- note added: "overvoltage protection"
- note added: "supply select"
- note added: "voltage level regulation"

Commit message: added ISO 9141 transceiver circuit
Parts:
- added IC6: LM339D, linear3:LM339D
- added R29, R30, R31, R32: 10k, rcl:R-EU_R0805
- added R33, R35: 510R 0W5, rcl:R-EU_R0805
- added R34, R36: 1k, rcl:R-EU_R0805
- added T4, T5: MMBT3904, transistor:MMBT3904LT1-NPN-SOT23-BEC
- T2: value (none) -> MMBT3904
Connections:
- new net N$35: IC6A.+IN, R29.2, R30.1
- new net N$36: IC6A.-IN, R31.2
- new net N$37: R34.2, T4.B
- new net N$38: R36.2, T5.B
- net !ISO_K_TX: now also R34.1
- net !ISO_L_TX: now also R36.1
- net !ISO_RX: now also IC6A.OUT, R32.2
- net +12V: now also IC6P.V+, R29.1, R33.1, R35.1
- net +3V3: now also R32.1
- net GND: now also IC6P.GND, R30.2, T4.E, T5.E
- net K_LINE: now also R31.1, R33.2, T4.C
- net L_LINE: now also R35.2, T5.C
Other:
- note added: "ISO 9141 / ISO 14230"
- moved on the sheet: D3, D4, D5, X1

Commit message: implemented CAN and SAE 1850 driver circuits
Parts:
- added C20, C21, C22: 1uF, rcl:C-EUC0805
- added C23: 100nF, rcl:C-EUC0805
- added D10, D11, D12: BAT54, diode:BAT54
- added H2: MOUNT-HOLE3.0, holes:MOUNT-HOLE3.0
- added IC7: LM317MSTT3, v-reg:LM317MSTT3
- added Q5: BSS84, transistor-small-signal:BSS84
- added Q6: BSS123, transistor-small-signal:BSS123
- added R37, R38: 100, rcl:R-EU_R0805
- added R39: 100k, rcl:R-EU_R0805
- added R40, R48: 240R, rcl:R-EU_R0805
- added R41: 866R, rcl:R-EU_R0805
- added R42: 374R, rcl:R-EU_R0805
- added R43, R44, R45, R46, R49, R51, R52, R53: 10k, rcl:R-EU_R0805
- added R47: 1k5, rcl:R-EU_R0805
- added R50: 2k7, rcl:R-EU_R0805
- added R54: 1k, rcl:R-EU_R0805
- added T6: 2N7002, zetex:NMOSSOT23
- added T7: BC847, transistor:BC847
- added U2: MCP2562-E/SN, MCP2562-E_SN:MCP2562-E/SN
Connections:
- removed net OBD_RX_LED: LED11.C
- removed net OBD_TX_LED: LED12.C
- removed net UART_RX_LED: LED9.C
- removed net UART_TX_LED: LED10.C
- new net N$39: C21.1, R38.1
- new net N$40: C20.1, R37.1
- new net N$41: IC7.ADJ, R40.1, R41.2
- new net N$42: R41.1, R42.2, T6.D
- new net N$43: R39.1, U2.STBY
- new net N$44: IC6C.+IN, R49.1
- new net N$45: IC6B.+IN, R43.1
- new net N$46: IC6B.-IN, R44.1
- new net N$47: D10.A, Q5.D
- new net N$48: IC6C.-IN, R50.2, R51.1
- new net N$49: D11.A, R46.1
- new net N$50: Q5.G, Q6.D, R47.1
- new net N$51: D12.C, R53.2
- new net N$53: R54.1, T7.B
- new net V_J1850: IC7.OUT, Q5.S, R40.2, R47.2
- net !J1850_BUS-_TX: now also R54.2
- net !OBD_RX_LED: now also LED11.C
- net !OBD_TX_LED: now also LED12.C
- net !UART_RX_LED: now also LED9.C
- net !UART_TX_LED: now also LED10.C
- net !VPW_RX: now also IC6C.OUT, R52.2
- net +12V: now also C23.1, IC7.IN
- net +3V3: now also R39.2, R45.1, R52.1, U2.VIO
- net +5V: now also C22.1, D12.A, R50.1, U2.VDD
- net CAN_RX: now also U2.RXD
- net CAN_TX: now also U2.TXD
- net GND: now also C20.2, C21.2, C22.2, C23.2, D11.C, Q6.S, R42.1, R48.1, R51.2, T6.S, T7.E, U2.VSS
- net HS_CAN_HI: now also R37.2, U2.CANH
- net HS_CAN_LO: now also R38.2, U2.CANL
- net J1850_BUS+: now also D10.C, R43.2, R46.2, R49.2
- net J1850_BUS+_TX: now also Q6.G, R48.2
- net J1850_BUS-: now also R44.2, R53.1, T7.C
- net PWM/!VPW: now also T6.G
- net PWM_RX: now also IC6B.OUT, R45.2
Other:
- note added: "High-Speed CAN"
- note added: "SAE J1850 VPW / PWM"
- note added: "STN1110 OBDII Translation"

Commit message: added k-line-adapter schematic and board finished first shot of qsd67lc_v2 schematic
Parts:
- removed C20, C21, C22: 1uF, rcl:C-EUC0805
- removed C23: 100nF, rcl:C-EUC0805
- removed D10, D11, D12: BAT54, diode:BAT54
- removed D3: PESD1CAN, diode:PESD1CAN
- removed D4, D5: BAS40-06, diode:BAS40-06
- removed IC6: LM339D, linear3:LM339D
- removed IC7: LM317MSTT3, v-reg:LM317MSTT3
- removed LED10, LED12: orange, led:LEDCHIP-LED0805
- removed LED11, LED9: yellow, led:LEDCHIP-LED0805
- removed Q5: BSS84, transistor-small-signal:BSS84
- removed Q6: BSS123, transistor-small-signal:BSS123
- removed R21, R22, R23, R24: 220R, rcl:R-EU_R0805
- removed R29, R30, R31, R32, R43, R44, R45, R46, R49, R51, R52, R53: 10k, rcl:R-EU_R0805
- removed R33, R35: 510R 0W5, rcl:R-EU_R0805
- removed R34, R36, R54: 1k, rcl:R-EU_R0805
- removed R37, R38: 100, rcl:R-EU_R0805
- removed R39: 100k, rcl:R-EU_R0805
- removed R40, R48: 240R, rcl:R-EU_R0805
- removed R41: 866R, rcl:R-EU_R0805
- removed R42: 374R, rcl:R-EU_R0805
- removed R47: 1k5, rcl:R-EU_R0805
- removed R50: 2k7, rcl:R-EU_R0805
- removed T4, T5: MMBT3904, transistor:MMBT3904LT1-NPN-SOT23-BEC
- removed T6: 2N7002, zetex:NMOSSOT23
- removed T7: BC847, transistor:BC847
- removed U2: MCP2562-E/SN, MCP2562-E_SN:MCP2562-E/SN
- removed X1: (no value), con-subd:M09HP
- added C24, C25, C26: 1uF, rcl:C-EUC0805
- added C27: 100nF, rcl:C-EUC0805
- added D13: PESD1CAN, diode:PESD1CAN
- added D14, D15: BAS40-06, diode:BAS40-06
- added D16, D17, D18: BAT54, diode:BAT54
- added IC10: LM317MSTT3, v-reg:LM317MSTT3
- added IC8, IC9: LM339D, linear3:LM339D
- added LED14, LED16: yellow, led:LEDCHIP-LED0805
- added LED15, LED17: orange, led:LEDCHIP-LED0805
- added Q7: BSS84, transistor-small-signal:BSS84
- added Q8: BSS123, transistor-small-signal:BSS123
- added R55, R56, R57, R58: 220R, rcl:R-EU_R0805
- added R59, R60, R61, R62, R73, R74, R75, R76, R79, R81, R82, R83: 10k, rcl:R-EU_R0805
- added R63, R65: 510R 0W5, rcl:R-EU_R0805
- added R64, R66, R84: 1k, rcl:R-EU_R0805
- added R67, R68: 100, rcl:R-EU_R0805
- added R69: 100k, rcl:R-EU_R0805
- added R70, R78: 240R, rcl:R-EU_R0805
- added R71: 866R, rcl:R-EU_R0805
- added R72: 374R, rcl:R-EU_R0805
- added R77: 1k5, rcl:R-EU_R0805
- added R80: 2k7, rcl:R-EU_R0805
- added T10: 2N7002, zetex:NMOSSOT23
- added T11: BC847, transistor:BC847
- added T8, T9: MMBT3904, transistor:MMBT3904LT1-NPN-SOT23-BEC
- added U3: MCP2562-E/SN, MCP2562-E_SN:MCP2562-E/SN
- added X2: (no value), con-subd:M09HP
- L1, L2: device rcl:L-EU2200-15.24 -> own_parts:L-LEU-09HCP
- R25: value 220R -> 330R
Connections:
- removed net N$26: LED12.A, R21.2
- removed net N$27: LED11.A, R22.2
- removed net N$28: LED10.A, R23.2
- removed net N$29: LED9.A, R24.2
- removed net N$35: IC6A.+IN, R29.2, R30.1
- removed net N$36: IC6A.-IN, R31.2
- removed net N$37: R34.2, T4.B
- removed net N$38: R36.2, T5.B
- removed net N$39: C21.1, R38.1
- removed net N$40: C20.1, R37.1
- removed net N$41: IC7.ADJ, R40.1, R41.2
- removed net N$42: R41.1, R42.2, T6.D
- removed net N$43: R39.1, U2.STBY
- removed net N$44: IC6C.+IN, R49.1
- removed net N$45: IC6B.+IN, R43.1
- removed net N$46: IC6B.-IN, R44.1
- removed net N$47: D10.A, Q5.D
- removed net N$48: IC6C.-IN, R50.2, R51.1
- removed net N$49: D11.A, R46.1
- removed net N$50: Q5.G, Q6.D, R47.1
- removed net N$51: D12.C, R53.2
- removed net N$53: R54.1, T7.B
- new net N$52: LED17.A, R55.2
- new net N$54: LED16.A, R56.2
- new net N$55: LED15.A, R57.2
- new net N$56: LED14.A, R58.2
- new net N$57: IC8A.+IN, R59.2, R60.1
- new net N$58: IC8A.-IN, R61.2
- new net N$59: R64.2, T8.B
- new net N$60: R66.2, T9.B
- new net N$61: C25.1, R68.1
- new net N$62: C24.1, R67.1
- new net N$63: R69.1, U3.STBY
- new net N$64: IC10.ADJ, R70.1, R71.2
- new net N$65: R71.1, R72.2, T10.D
- new net N$66: IC9B.+IN, R73.1
- new net N$67: IC9B.-IN, R74.1
- new net N$68: D16.A, Q7.D
- new net N$69: D17.A, R76.1
- new net N$70: Q7.G, Q8.D, R77.1
- new net N$71: IC9C.+IN, R79.1
- new net N$72: IC9C.-IN, R80.2, R81.1
- new net N$73: D18.C, R83.2
- new net N$74: R84.1, T11.B
- net !ISO_K_TX: now also R64.1; no longer R34.1
- net !ISO_L_TX: now also R66.1; no longer R36.1
- net !ISO_RX: now also IC8A.OUT, R62.2; no longer IC6A.OUT, R32.2
- net !J1850_BUS-_TX: now also R84.2; no longer R54.2
- net !OBD_RX_LED: now also LED16.C; no longer LED11.C
- net !OBD_TX_LED: now also LED17.C; no longer LED12.C
- net !UART_RX_LED: now also LED14.C; no longer LED9.C
- net !UART_TX_LED: now also LED15.C; no longer LED10.C
- net !VPW_RX: now also IC9C.OUT, R82.2; no longer IC6C.OUT, R52.2
- net +12V: now also C27.1, IC10.IN, IC8P.V+, R59.1, R63.1, R65.1; no longer C23.1, IC2.VBB, IC6P.V+, IC7.IN, Q2.D, R29.1, R33.1, R35.1
- net +3V3: now also R55.1, R56.1, R57.1, R58.1, R62.1, R69.2, R75.1, R82.1, U3.VIO; no longer R21.1, R22.1, R23.1, R24.1, R32.1, R39.2, R45.1, R52.1, U2.VIO
- net +5V: now also C26.1, D18.A, R80.1, U3.VDD; no longer C22.1, D12.A, R50.1, U2.VDD
- net CAN_RX: now also U3.RXD; no longer U2.RXD
- net CAN_TX: now also U3.TXD; no longer U2.TXD
- net GND: now also C24.2, C25.2, C26.2, C27.2, D13.1, D13.3, D14.AA, D15.AA, D17.C, IC8P.GND, Q8.S, R60.2, R72.1, R78.1, R81.2, T10.S, T11.E, T8.E, T9.E, U3.VSS, X2.1, X2.2; no longer C20.2, C21.2, C22.2, C23.2, D11.C, D3.1, D3.3, D4.AA, D5.AA, IC6P.GND, Q6.S, R30.2, R42.1, R48.1, R51.2, T4.E, T5.E, T6.S, T7.E, U2.VSS, X1.1, X1.2
- net HS_CAN_HI: now also R67.2, U3.CANH, X2.3; no longer R37.2, U2.CANH, X1.3
- net HS_CAN_LO: now also D13.2, R68.2, U3.CANL, X2.5; no longer D3.2, R38.2, U2.CANL, X1.5
- net J1850_BUS+: now also D15.K2, D16.C, R73.2, R76.2, R79.2, X2.7; no longer D10.C, D5.K2, R43.2, R46.2, R49.2, X1.7
- net J1850_BUS+_TX: now also Q8.G, R78.2; no longer Q6.G, R48.2
- net J1850_BUS-: now also D15.K1, R74.2, R83.1, T11.C, X2.6; no longer D5.K1, R44.2, R53.1, T7.C, X1.6
- net KL15: now also IC2.VBB, Q2.D
- net KL30: now also X2.9; no longer X1.9
- net K_LINE: now also D14.K2, R61.1, R63.2, T8.C, X2.4; no longer D4.K2, R31.1, R33.2, T4.C, X1.4
- net L_LINE: now also D14.K1, R65.2, T9.C, X2.8; no longer D4.K1, R35.2, T5.C, X1.8
- net PWM/!VPW: now also T10.G; no longer T6.G
- net PWM_RX: now also IC9B.OUT, R75.2; no longer IC6B.OUT, R45.2
- net V_J1850: now also IC10.OUT, Q7.S, R70.2, R77.2; no longer IC7.OUT, Q5.S, R40.2, R47.2

Commit message: working on kline adapter ...
Parts:
- removed IC8: LM339D, linear3:LM339D
- removed T10: 2N7002, zetex:NMOSSOT23
- added Q5: BSS123, transistor-small-signal:BSS123
- C13: device rcl:CPOL-EUE5-10.5 -> rcl:CPOL-EUE2-5
- C14, C9: device rcl:CPOL-EUE5-13 -> rcl:CPOL-EUE5-10.5
- D2: value BZX55C3V3 -> 3V3; device diode:BZX55 -> diode:ZENER-DIODESOD80C
- D8, D9: value (none) -> 18V; device diode:ZENER-DIODESMB -> diode:ZENER-DIODESOD80C
- Q1: device crystal:CRYSTALHC18U-V -> crystal:CRYSTALHC49U-V
- Q3: device crystal:CRYSTALHC49U70 -> crystal:CRYSTALHC49U-V
- Q4: value IRLML5203 -> IRF7424; device transistor-power:IRLML5203 -> transistor-fet:BSO201SP
- R26, R28: value (none) -> 100k
- R27: value (none) -> 10k
- R63, R65: device rcl:R-EU_R0805 -> rcl:R-EU_0207/12
- R67, R68: value 100 -> 100R
- R71: value 866R -> 1k
- R72: value 374R -> 430R
- T2: device transistor:MMBT3906LT1-PNP-SOT23-BEC -> transistor:BC807-16-PNP-SOT23-BEC
- T9: device transistor:MMBT3904LT1-NPN-SOT23-BEC -> transistor:BC817-16-NPN-SOT23-BEC
Connections:
- net !ISO_RX: now also IC9A.OUT; no longer IC8A.OUT
- net +12V: now also IC9P.V+; no longer IC8P.V+
- net GND: now also IC9P.GND, Q5.S; no longer IC8P.GND, T10.S
- net N$57: now also IC9A.+IN; no longer IC8A.+IN
- net N$58: now also IC9A.-IN; no longer IC8A.-IN
- net N$65: now also Q5.D; no longer T10.D
- net PWM/!VPW: now also Q5.G; no longer T10.G
